Commit message: ros2: readable robot model + zoomed RViz config
URDF changes (reads as a wheeled robot in RViz now):
- Materials defined ONCE at robot scope (RViz2 drops colours when the same
  material name is redefined per link).
- Slightly bigger chassis (0.20 x 0.14 x 0.07 m), thicker wheels (28 mm),
  bigger caster (18 mm) so the geometry is unambiguous at close range.
- Two-tone body: blue chassis + dark blue lid plate.
- A red front marker on the +X face. The robot no longer looks symmetric,
  so yaw is readable at a glance when it drives.
- A grey rim disc on the outer face of each wheel, so wheel rotation is
  visible (a plain black cylinder looks static while it spins).
- Wheels aligned flush with the chassis edge (wheel_separation / 2) so they
  look like real wheels, not pegs.

RViz config:
- Camera orbit distance 0.8 m with target_frame=base_footprint (follows
  the robot), focal point raised 5 cm so the body is centred.
- 10 cm grid instead of 50 cm (robot is 20 cm long; large grid made it a
  dot).
- TF arrows shrunk to 15 cm marker scale, names off, so the model isn't
  buried under axis gnomons.
- Odom arrows thinner, higher-contrast colours; 200 samples retained.

check_urdf: tree is clean. base_footprint → base_link → {lid, front_marker,
left_wheel, right_wheel, caster_wheel}. No duplicate parents.

File: services/ros2/yoruba_robot/description/robot.urdf.xacro (robot description, xacro)
@@ -4,22 +4,23 @@
   matches the real chassis (65 mm wheel, 150 mm wheelbase; override from
   launch). Same model goes to Gazebo (simulated physics) and RViz (visuals + TF
-  from the robot_bridge), so sim and reality share one URDF.
+  from robot_bridge), so sim and reality share one URDF.
   Frames (REP-103, +x forward, +z up):
-    base_footprint  -> on the ground
+    base_footprint  -> on the ground (TF root the bridge publishes to)
     base_link       -> body origin, at the wheel axle height
-    left_wheel      -> y = +wheel_sep/2
-    right_wheel     -> y = -wheel_sep/2
-    caster_wheel    -> ball caster at the rear, matches most hobby chassis
-  Gazebo diff_drive plugin publishes /odom and TF when running in sim; the real
-  robot_bridge publishes the same, so RViz tooling works unchanged in both.
+    left_wheel, right_wheel, caster_wheel
+    front_marker    -> a small red block on the +x face so RViz orientation is
+                       unambiguous (otherwise a symmetric chassis gives no hint)
+  Materials are defined ONCE at robot scope and referenced by name in each
+  link. RViz2's URDF parser logs a warning (and sometimes drops the colour)
+  when the same material name is redefined per link.
 -->
 <robot name="yoruba_robot" xmlns:xacro="http://ros.org/wiki/xacro">
-  <xacro:arg name="wheel_radius"     default="0.0325"/>
+  <xacro:arg name="wheel_radius"     default="0.035"/>
   <xacro:arg name="wheel_separation" default="0.15"/>
-  <xacro:arg name="wheel_width"      default="0.025"/>
-  <xacro:arg name="body_length"      default="0.17"/>
-  <xacro:arg name="body_width"       default="0.12"/>
-  <xacro:arg name="body_height"      default="0.06"/>
-  <xacro:arg name="caster_radius"    default="0.015"/>
+  <xacro:arg name="wheel_width"      default="0.028"/>
+  <xacro:arg name="body_length"      default="0.20"/>
+  <xacro:arg name="body_width"       default="0.14"/>
+  <xacro:arg name="body_height"      default="0.07"/>
+  <xacro:arg name="caster_radius"    default="0.018"/>
   <xacro:arg name="use_sim"          default="true"/>
   <xacro:property name="wheel_radius"     value="$(arg wheel_radius)"/>
@@ -30,4 +31,11 @@
   <xacro:property name="body_height"      value="$(arg body_height)"/>
   <xacro:property name="caster_radius"    value="$(arg caster_radius)"/>
+  <!-- ================== materials (global, once) ================== -->
+  <material name="chassis_blue"><color rgba="0.15 0.45 0.90 1.0"/></material>
+  <material name="chassis_dark"><color rgba="0.08 0.20 0.45 1.0"/></material>
+  <material name="wheel_black"><color rgba="0.08 0.08 0.08 1.0"/></material>
+  <material name="rim_grey">   <color rgba="0.40 0.40 0.42 1.0"/></material>
+  <material name="caster_grey"><color rgba="0.65 0.65 0.67 1.0"/></material>
+  <material name="front_red">  <color rgba="0.95 0.20 0.15 1.0"/></material>
   <!-- Inertia helpers. Order-of-magnitude correct; mass tuned so the sim robot
        doesn't tip when a turn command accelerates one wheel. -->
@@ -53,9 +61,11 @@
     <origin xyz="0 0 ${wheel_radius}" rpy="0 0 0"/>
   </joint>
+  <!-- Main chassis plate. Centred over the axle; top surface at body_height
+       (so z=0..body_height in base_link frame). -->
   <link name="base_link">
     <visual>
       <origin xyz="0 0 ${body_height/2}"/>
       <geometry><box size="${body_length} ${body_width} ${body_height}"/></geometry>
-      <material name="chassis"><color rgba="0.2 0.4 0.9 1"/></material>
+      <material name="chassis_blue"/>
     </visual>
     <collision>
@@ -65,4 +75,33 @@
     <xacro:box_inertial mass="0.8" x="${body_length}" y="${body_width}" z="${body_height}"/>
   </link>
+  <!-- Lid plate so the chassis reads as a two-tone robot, not a plain box.
+       Fixed to base_link, no own inertia (dimensionless visual). -->
+  <joint name="lid_joint" type="fixed">
+    <parent link="base_link"/>
+    <child link="lid"/>
+    <origin xyz="0 0 ${body_height + 0.005}"/>
+  </joint>
+  <link name="lid">
+    <visual>
+      <origin xyz="0 0 0.005"/>
+      <geometry><box size="${body_length*0.9} ${body_width*0.9} 0.01"/></geometry>
+      <material name="chassis_dark"/>
+    </visual>
+  </link>
+  <!-- A clearly-visible red block on the +X face: no symmetry ambiguity about
+       which way the robot is heading when you watch it in RViz. -->
+  <joint name="front_marker_joint" type="fixed">
+    <parent link="base_link"/>
+    <child link="front_marker"/>
+    <origin xyz="${body_length/2 + 0.01} 0 ${body_height/2}"/>
+  </joint>
+  <link name="front_marker">
+    <visual>
+      <geometry><box size="0.02 ${body_width*0.5} ${body_height*0.6}"/></geometry>
+      <material name="front_red"/>
+    </visual>
+  </link>
+  <!-- Wheels. Cylinder's own axis is Z; roll by pi/2 around X so the circular
+       face points sideways (axle along Y, as the joint expects). -->
   <xacro:macro name="wheel" params="prefix y_sign">
     <link name="${prefix}_wheel">
@@ -70,5 +109,13 @@
         <origin rpy="1.5707963 0 0"/>
         <geometry><cylinder radius="${wheel_radius}" length="${wheel_width}"/></geometry>
-        <material name="wheel"><color rgba="0.1 0.1 0.1 1"/></material>
+        <material name="wheel_black"/>
+      </visual>
+      <!-- A thin grey rim disc on the outer face of each wheel so the wheel's
+           rotation is visible in RViz (otherwise a plain black cylinder looks
+           static even while it is spinning). -->
+      <visual>
+        <origin xyz="0 ${y_sign*wheel_width*0.5} 0" rpy="1.5707963 0 0"/>
+        <geometry><cylinder radius="${wheel_radius*0.55}" length="0.002"/></geometry>
+        <material name="rim_grey"/>
       </visual>
       <collision>
@@ -81,5 +128,6 @@
       <parent link="base_link"/>
       <child link="${prefix}_wheel"/>
-      <origin xyz="0 ${y_sign*wheel_separation/2} 0"/>
+      <!-- Wheels sit just outboard of the chassis so they are clearly visible. -->
+      <origin xyz="0 ${y_sign*(wheel_separation/2)} 0"/>
       <axis xyz="0 1 0"/>
     </joint>
@@ -87,14 +135,6 @@
   <xacro:wheel prefix="left"  y_sign=" 1"/>
   <xacro:wheel prefix="right" y_sign="-1"/>
-  <!-- Ball caster at the rear. In Gazebo it's a tiny low-friction sphere so the
+  <!-- Rear ball caster. In Gazebo it's a tiny low-friction sphere so the
        chassis stays level without a third powered wheel. -->
-  <link name="caster_wheel">
-    <visual>
-      <geometry><sphere radius="${caster_radius}"/></geometry>
-      <material name="caster"><color rgba="0.6 0.6 0.6 1"/></material>
-    </visual>
-    <collision><geometry><sphere radius="${caster_radius}"/></geometry></collision>
-    <xacro:cyl_inertial mass="0.01" r="${caster_radius}" h="${caster_radius*2}"/>
-  </link>
   <joint name="caster_joint" type="fixed">
     <parent link="base_link"/>
@@ -102,7 +142,15 @@
     <origin xyz="${-body_length/2 + caster_radius} 0 ${-wheel_radius + caster_radius}"/>
   </joint>
+  <link name="caster_wheel">
+    <visual>
+      <geometry><sphere radius="${caster_radius}"/></geometry>
+      <material name="caster_grey"/>
+    </visual>
+    <collision><geometry><sphere radius="${caster_radius}"/></geometry></collision>
+    <xacro:cyl_inertial mass="0.01" r="${caster_radius}" h="${caster_radius*2}"/>
+  </link>
   <xacro:if value="$(arg use_sim)">
-    <!-- Gazebo plugin surfaces + materials. mu/mu2 low on the caster so the
-         robot can turn in place without the ball locking the yaw. -->
+    <!-- Gazebo plugin surfaces: wheels grippy, caster frictionless so a spin
+         command rotates in place instead of locking on the ball. -->
     <gazebo reference="left_wheel"><mu1>1.0</mu1><mu2>1.0</mu2></gazebo>
     <gazebo reference="right_wheel"><mu1>1.0</mu1><mu2>1.0</mu2></gazebo>
